Commit message: nav2 on real robot

File: description/robot_core.xacro (robot description, xacro)
@@ -86,5 +86,5 @@
         <child link="right_wheel"/>
         <origin xyz="0 -0.1775 0" rpy="${pi/2} 0 0" />
-        <axis xyz="0 0 -1"/>
+        <axis xyz="0 0 1"/>
     </joint>
     <link name="right_wheel">
